File: 1_first/STM32F103C8T6_Minimal_v1/STM32F103C8T6_Minimal_v1.kicad_sch (KiCad schematic)
At the start: 0 parts

Commit message: Added USB B micro connector
Other:
- title: (none) -> Basic STM32
Changed lines of the file:
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@@
 	(generator_version "10.0")
 	(paper "A4")
+	(title_block
+		(title "Basic STM32")
+		(date "2026-05-18")
+		(rev "0.1")
+	)
 	(sheet
 		(at 3.81 508)
